Commit message: change panda urdf

File: src/curobo/content/assets/robot/franka_description/franka_panda.urdf (robot description, URDF)
Before this commit: robot panda, 15 links, 14 joints
Joints:
- joint panda_hand_joint: origin xyz=0 0 0 rpy=0 0 -0.785398163397 -> xyz=0 0 0.1034 rpy=0 0 -0.785398163397
